Commit message: feat: add welding cell (table + robot pedestal) recreated from real BEAM cell
- welding_cell.xacro: System-28 style welding table (2.0x1.0 m, work
  surface 0.87 m) + 0.4x0.4x0.3 m robot pedestal riser on the rear edge;
  all dimensions parametrized (estimated from photo via 100 mm hole grid)
- robot mounts on pedestal_mount (base at z=1.17 m); welding_cell:=false
  keeps the bare robot on the floor
- SRDF collision exceptions for base/pedestal/table
- spawn z 0.05 -> 0.0; removed red demo cylinder from the world

Co-Authored-By: Claude Fable 5 <noreply@anthropic.com>

File: urdf/crx10ia_gz.urdf.xacro (robot description, xacro)
@@ -2,13 +2,24 @@
 <robot xmlns:xacro="http://wiki.ros.org/xacro" name="crx10ia">
   <xacro:arg name="simulation_controllers" default="" />
+  <!-- welding cell (table + robot pedestal); set to false for a bare robot on the floor -->
+  <xacro:arg name="welding_cell" default="true" />
   <xacro:include filename="$(find fanuc_crx_description)/urdf/crx10ia_urdf_macro.xacro"/>
   <xacro:include filename="$(find fanuc_gazebo)/urdf/crx_gz_ros2_control_macro.xacro"/>
   <xacro:include filename="$(find fanuc_gazebo)/urdf/welding_torch.xacro"/>
   <xacro:include filename="$(find fanuc_gazebo)/urdf/include/fanuc_oak_d_pro_w_macros.xacro"/>
+  <xacro:include filename="$(find fanuc_gazebo)/urdf/welding_cell.xacro"/>
   <link name="world"/>
   <link name="end_effector"/>
-  <xacro:crx10ia parent="world" child="end_effector" prefix="">
-    <origin xyz="0 0 0" rpy="0 0 0"/>
-  </xacro:crx10ia>
+  <xacro:if value="$(arg welding_cell)">
+    <xacro:welding_cell parent="world" prefix=""/>
+    <xacro:crx10ia parent="pedestal_mount" child="end_effector" prefix="">
+      <origin xyz="0 0 0" rpy="0 0 0"/>
+    </xacro:crx10ia>
+  </xacro:if>
+  <xacro:unless value="$(arg welding_cell)">
+    <xacro:crx10ia parent="world" child="end_effector" prefix="">
+      <origin xyz="0 0 0" rpy="0 0 0"/>
+    </xacro:crx10ia>
+  </xacro:unless>
   <xacro:crx_welding_torch parent="end_effector" prefix=""/>
   <xacro:fanuc_mount_oak_d_pro_w parent_link="J6_link" simulation="true" oak_gazebo_rgbd_sensor="true"/>

Commit message: feat: add FANUC hybrid RealSense launch and sim-time stamp sync
Hybrid cell keeps the driver on wall time and republishes camera topics
from /clock, plus OAK-SR frame macros and related sim/real launch wiring.

Co-authored-by: Cursor <cursoragent@cursor.com>

File: urdf/crx10ia_gz.urdf.xacro (robot description, xacro)
@@ -4,8 +4,16 @@
   <!-- welding cell (table + robot pedestal); set to false for a bare robot on the floor -->
   <xacro:arg name="welding_cell" default="true" />
+  <!-- gazebo_oak | realsense_d435 | none (hybrid: real cam + identity static TF) -->
+  <xacro:arg name="wrist_camera" default="gazebo_oak" />
+  <xacro:property name="wrist_camera_selected" value="$(arg wrist_camera)"/>
   <xacro:include filename="$(find fanuc_crx_description)/urdf/crx10ia_urdf_macro.xacro"/>
   <xacro:include filename="$(find seam_ros2_pkg)/urdf/crx_gz_ros2_control_macro.xacro"/>
   <xacro:include filename="$(find seam_ros2_pkg)/urdf/welding_torch.xacro"/>
-  <xacro:include filename="$(find seam_ros2_pkg)/urdf/include/fanuc_oak_d_pro_w_macros.xacro"/>
+  <xacro:if value="${wrist_camera_selected == 'gazebo_oak'}">
+    <xacro:include filename="$(find seam_ros2_pkg)/urdf/include/fanuc_oak_d_pro_w_macros.xacro"/>
+  </xacro:if>
+  <xacro:if value="${wrist_camera_selected == 'realsense_d435'}">
+    <xacro:include filename="$(find seam_ros2_pkg)/urdf/include/fanuc_realsense_d435_handeye_macros.xacro"/>
+  </xacro:if>
   <xacro:include filename="$(find seam_ros2_pkg)/urdf/welding_cell.xacro"/>
   <link name="world"/>
@@ -23,5 +31,10 @@
   </xacro:unless>
   <xacro:crx_welding_torch parent="end_effector" prefix=""/>
-  <xacro:fanuc_mount_oak_d_pro_w parent_link="J6_link" simulation="true" oak_gazebo_rgbd_sensor="true"/>
+  <xacro:if value="${wrist_camera_selected == 'gazebo_oak'}">
+    <xacro:fanuc_mount_oak_d_pro_w parent_link="J6_link" simulation="true" oak_gazebo_rgbd_sensor="true"/>
+  </xacro:if>
+  <xacro:if value="${wrist_camera_selected == 'realsense_d435'}">
+    <xacro:fanuc_mount_realsense_d435_handeye parent_link="J6_link" use_mesh="true"/>
+  </xacro:if>
   <xacro:crx_gz_control name="crx10ia" prefix=""/>
   <gazebo reference="base_link">

File: urdf/crx10ia_real.urdf.xacro (robot description, xacro)
@@ -1,5 +1,7 @@
 <?xml version="1.0"?>
 <!--
-  Physical FANUC CRX-10iA + ROBO WH-PP W500 torch + RealSense D435.
+  Physical FANUC CRX-10iA + ROBO WH-PP W500 torch + wrist camera.
+  camera_model: realsense_d435 | oak_d_pro_w | oak_sr
+  Camera driver is launched separately; URDF owns TF (driver publish_tf off).
   Uses fanuc_hardware_interface ros2_control (Stream Motion / mock).
   Gazebo plugins are intentionally omitted.
@@ -17,8 +19,18 @@
   <xacro:arg name="welding_cell" default="true"/>
   <xacro:arg name="prefix" default=""/>
+  <xacro:arg name="camera_model" default="realsense_d435"/>
+  <xacro:property name="camera_model_selected" value="$(arg camera_model)"/>
   <xacro:include filename="$(find fanuc_crx_description)/urdf/crx10ia_urdf_macro.xacro"/>
   <xacro:include filename="$(find seam_ros2_pkg)/urdf/welding_torch.xacro"/>
-  <xacro:include filename="$(find seam_ros2_pkg)/urdf/include/fanuc_realsense_d435_handeye_macros.xacro"/>
   <xacro:include filename="$(find seam_ros2_pkg)/urdf/welding_cell.xacro"/>
+  <xacro:if value="${camera_model_selected == 'realsense_d435'}">
+    <xacro:include filename="$(find seam_ros2_pkg)/urdf/include/fanuc_realsense_d435_handeye_macros.xacro"/>
+  </xacro:if>
+  <xacro:if value="${camera_model_selected == 'oak_d_pro_w'}">
+    <xacro:include filename="$(find seam_ros2_pkg)/urdf/include/fanuc_oak_d_pro_w_macros.xacro"/>
+  </xacro:if>
+  <xacro:if value="${camera_model_selected == 'oak_sr'}">
+    <xacro:include filename="$(find seam_ros2_pkg)/urdf/include/fanuc_oak_d_sr_handeye_macros.xacro"/>
+  </xacro:if>
   <xacro:if value="$(arg use_mock)">
     <xacro:include filename="$(find fanuc_hardware_interface)/config/crx_mock_ros2_control_macro.xacro"/>
@@ -41,5 +53,13 @@
   </xacro:unless>
   <xacro:crx_welding_torch parent="end_effector" prefix=""/>
-  <xacro:fanuc_mount_realsense_d435_handeye parent_link="J6_link" use_mesh="true"/>
+  <xacro:if value="${camera_model_selected == 'realsense_d435'}">
+    <xacro:fanuc_mount_realsense_d435_handeye parent_link="J6_link" use_mesh="true"/>
+  </xacro:if>
+  <xacro:if value="${camera_model_selected == 'oak_d_pro_w'}">
+    <xacro:fanuc_mount_oak_d_pro_w parent_link="J6_link" simulation="false"/>
+  </xacro:if>
+  <xacro:if value="${camera_model_selected == 'oak_sr'}">
+    <xacro:fanuc_mount_oak_d_sr_handeye parent_link="J6_link" simulation="false" oak_visual_mesh="true"/>
+  </xacro:if>
   <xacro:crx_control name="crx10ia" prefix="$(arg prefix)"/>
 </robot>

File: urdf/include/fanuc_realsense_d435_handeye_macros.xacro (robot description, xacro)
@@ -6,8 +6,9 @@
   Do NOT run rs_launch.py with publish_tf true. robot_state_publisher owns
   the camera TF tree via this macro.
-  PLACEHOLDER mount (rough, copied from the sim OAK mid-gun pose). After site
-  hand-eye calibration, bake the result with hand_eye_calibration.realsense_mount_cli
-  (joint name fanuc_j6_realsense_d435_mount), then rebuild seam_ros2_pkg and
-  restart the stack.
+    PLACEHOLDER mount intentionally reuses the FANUC OAK-D Pro W mid-gun pose
+  (same xyz/rpy as fanuc_oak_d_pro_w_macros.xacro). Optical frame names still
+  match realsense2_camera (camera_color_optical_frame, …). After site hand-eye,
+  bake with hand_eye_calibration.realsense_mount_cli
+  (joint name fanuc_j6_realsense_d435_mount), then rebuild seam_ros2_pkg.
 -->
 <robot xmlns:xacro="http://ros.org/wiki/xacro" name="fanuc_realsense_d435_attachment_defs">
@@ -16,5 +17,5 @@
     <link name="fanuc_realsense_mount"/>
     <joint name="fanuc_j6_realsense_d435_mount" type="fixed">
-      <!-- PLACEHOLDER: replace after hand-eye (see file header). -->
+      <!-- OAK mid-gun mount (fanuc_oak_d_pro_w); fine until site hand-eye. -->
       <origin
         xyz="0.300000000000 0.000000000000 0.130000000000"

Commit message: feat(sim): add CRX wrist RGB-D sensors and calibrated Gazebo URDF
- add fanuc_gz_rgbd_bridge.yaml and Femto Bolt / RGB-D sensor xacro macros for simulated wrist cameras
- load the calibration store mount and TCP in crx10ia_gz.urdf.xacro and crx_gz_sim_moveit.launch.py
- update srdf, kinematics, welding_torch.xacro and package.xml
- add meshes/cylinder_flat_m.stl workpiece mesh

Co-Authored-By: Claude Opus 5.5 <noreply@anthropic.com>

File: urdf/crx10ia_gz.urdf.xacro (robot description, xacro)
@@ -2,10 +2,25 @@
 <robot xmlns:xacro="http://wiki.ros.org/xacro" name="crx10ia">
   <xacro:arg name="simulation_controllers" default="" />
-  <!-- welding cell (table + robot pedestal); set to false for a bare robot on the floor -->
+  <!-- welding cell; set to false for a bare robot on the floor.
+       crx10ia_l: digital twin of the real cell (crx_description crx10ia_l_cell.xacro, same as
+       the real bringup); crx10ia: older estimate in welding_cell.xacro -->
   <xacro:arg name="welding_cell" default="true" />
-  <!-- gazebo_oak | realsense_d435 | none (hybrid: real cam + identity static TF) -->
+  <!-- gazebo_oak | gazebo_realsense | femto_bolt | realsense_d435 | none
+       (realsense_d435: TF only; none: hybrid real cam + identity static TF) -->
   <xacro:arg name="wrist_camera" default="gazebo_oak" />
   <xacro:property name="wrist_camera_selected" value="$(arg wrist_camera)"/>
-  <xacro:include filename="$(find fanuc_crx_description)/urdf/crx10ia_urdf_macro.xacro"/>
+  <!-- crx10ia | crx10ia_l (fanuc_crx_description macros share link/joint names) -->
+  <xacro:arg name="model" default="crx10ia" />
+  <xacro:property name="model" value="$(arg model)"/>
+  <xacro:property name="gz_rgbd_camera" value="${wrist_camera_selected in ('gazebo_realsense', 'femto_bolt')}"/>
+  <!-- Femto / D435 mount (flange -> camera root, `nominal` origin) and welding TCP (flange ->
+       welding_tcp, `sim` origin) from the calibration store, same files and format as the
+       real crx_description robot (crx_calibration_args.xacro). GUI launches pass the
+       robot's active ~/.ros/calibration/<model>/... current.yaml; '' = crx_description default. -->
+  <xacro:arg name="camera_calibration" default="" />
+  <xacro:arg name="tcp_calibration" default="" />
+  <xacro:property name="store_camera" value="${'femto_bolt' if wrist_camera_selected == 'femto_bolt' else ('realsense_d435' if wrist_camera_selected in ('gazebo_realsense', 'realsense_d435') else '')}"/>
+  <xacro:property name="tcp_sim_origin" value="${xacro.load_yaml('$(arg tcp_calibration)' or '$(find crx_description)/config/calibration/welding_tcp_default.yaml')['sim']}"/>
+  <xacro:include filename="$(find fanuc_crx_description)/urdf/${model}_urdf_macro.xacro"/>
   <xacro:include filename="$(find seam_ros2_pkg)/urdf/crx_gz_ros2_control_macro.xacro"/>
   <xacro:include filename="$(find seam_ros2_pkg)/urdf/welding_torch.xacro"/>
@@ -13,27 +28,56 @@
     <xacro:include filename="$(find seam_ros2_pkg)/urdf/include/fanuc_oak_d_pro_w_macros.xacro"/>
   </xacro:if>
-  <xacro:if value="${wrist_camera_selected == 'realsense_d435'}">
-    <xacro:include filename="$(find seam_ros2_pkg)/urdf/include/fanuc_realsense_d435_handeye_macros.xacro"/>
+  <xacro:if value="${store_camera != ''}">
+    <xacro:include filename="$(find crx_description)/urdf/include/crx_wrist_camera.xacro"/>
   </xacro:if>
-  <xacro:include filename="$(find seam_ros2_pkg)/urdf/welding_cell.xacro"/>
+  <xacro:if value="${gz_rgbd_camera}">
+    <xacro:include filename="$(find seam_ros2_pkg)/urdf/include/fanuc_gz_rgbd_sensors.xacro"/>
+  </xacro:if>
+  <xacro:property name="crx10ia_l_cell" value="${model == 'crx10ia_l'}"/>
+  <xacro:if value="${crx10ia_l_cell}">
+    <xacro:include filename="$(find crx_description)/urdf/crx10ia_l/crx10ia_l_cell.xacro"/>
+  </xacro:if>
+  <xacro:unless value="${crx10ia_l_cell}">
+    <xacro:include filename="$(find seam_ros2_pkg)/urdf/welding_cell.xacro"/>
+  </xacro:unless>
   <link name="world"/>
   <link name="end_effector"/>
   <xacro:if value="$(arg welding_cell)">
-    <xacro:welding_cell parent="world" prefix=""/>
-    <xacro:crx10ia parent="pedestal_mount" child="end_effector" prefix="">
-      <origin xyz="0 0 0" rpy="0 0 0"/>
-    </xacro:crx10ia>
+    <xacro:if value="${crx10ia_l_cell}">
+      <!-- world = floor; the cell hangs below base_link -->
+      <xacro:call macro="${model}" parent="world" child="end_effector" prefix="">
+        <origin xyz="0 0 ${crx10ia_l_cell_table_top_height + crx10ia_l_cell_pedestal_above_table}" rpy="0 0 0"/>
+      </xacro:call>
+      <xacro:crx10ia_l_cell parent="base_link"/>
+    </xacro:if>
+    <xacro:unless value="${crx10ia_l_cell}">
+      <xacro:welding_cell parent="world" prefix=""/>
+      <xacro:call macro="${model}" parent="pedestal_mount" child="end_effector" prefix="">
+        <origin xyz="0 0 0" rpy="0 0 0"/>
+      </xacro:call>
+    </xacro:unless>
   </xacro:if>
   <xacro:unless value="$(arg welding_cell)">
-    <xacro:crx10ia parent="world" child="end_effector" prefix="">
+    <xacro:call macro="${model}" parent="world" child="end_effector" prefix="">
       <origin xyz="0 0 0" rpy="0 0 0"/>
-    </xacro:crx10ia>
+    </xacro:call>
   </xacro:unless>
-  <xacro:crx_welding_torch parent="end_effector" prefix=""/>
+  <xacro:crx_welding_torch parent="end_effector" prefix=""
+                           tcp_parent="flange" tcp_xyz="${tcp_sim_origin['xyz']}" tcp_rpy="${tcp_sim_origin['rpy']}"/>
   <xacro:if value="${wrist_camera_selected == 'gazebo_oak'}">
     <xacro:fanuc_mount_oak_d_pro_w parent_link="J6_link" simulation="true" oak_gazebo_rgbd_sensor="true"/>
   </xacro:if>
-  <xacro:if value="${wrist_camera_selected == 'realsense_d435'}">
-    <xacro:fanuc_mount_realsense_d435_handeye parent_link="J6_link" use_mesh="true"/>
+  <xacro:if value="${store_camera != ''}">
+    <xacro:crx_wrist_camera camera="${store_camera}" parent_link="flange" nominal="true"
+      calibration_file="${'$(arg camera_calibration)' or '$(find crx_description)/config/calibration/' + store_camera + '_handeye_default.yaml'}"/>
+  </xacro:if>
+  <xacro:if value="${gz_rgbd_camera}">
+    <xacro:fanuc_wrist_rgbd_sensors camera="${wrist_camera_selected}"/>
+    <!-- Keep the FANUC sim camera frame API (oak_rgb_camera_optical_frame) the GUI uses. -->
+    <link name="oak_rgb_camera_optical_frame"/>
+    <joint name="fanuc_sim_optical_alias" type="fixed">
+      <parent link="camera_color_optical_frame"/>
+      <child link="oak_rgb_camera_optical_frame"/>
+    </joint>
   </xacro:if>
   <xacro:crx_gz_control name="crx10ia" prefix=""/>

File: urdf/welding_torch.xacro (robot description, xacro)
@@ -1,5 +1,7 @@
 <?xml version="1.0"?>
 <robot xmlns:xacro="http://wiki.ros.org/xacro">
-  <xacro:macro name="crx_welding_torch" params="parent prefix:=''">
+  <!-- tcp_parent/tcp_xyz/tcp_rpy: calibrated welding_tcp (crx10ia_gz: flange + store `sim`
+       origin); empty keeps the nominal Torch.stl wire tip on welding_torch. -->
+  <xacro:macro name="crx_welding_torch" params="parent prefix:='' tcp_parent:='' tcp_xyz:='' tcp_rpy:=''">
     <material name="${prefix}torch_metal">
       <color rgba="0.42 0.44 0.46 1.0"/>
@@ -38,6 +40,12 @@
     <link name="${prefix}welding_tcp"/>
     <joint name="${prefix}welding_tcp_joint" type="fixed">
-      <origin xyz="0.40642358 -0.01193078 0" rpy="0 0 0"/>
-      <parent link="${prefix}welding_torch"/>
+      <xacro:if value="${tcp_parent == ''}">
+        <origin xyz="0.40642358 -0.01193078 0" rpy="0 0 0"/>
+        <parent link="${prefix}welding_torch"/>
+      </xacro:if>
+      <xacro:unless value="${tcp_parent == ''}">
+        <origin xyz="${tcp_xyz}" rpy="${tcp_rpy}"/>
+        <parent link="${tcp_parent}"/>
+      </xacro:unless>
       <child link="${prefix}welding_tcp"/>
     </joint>
